File: board/spark.kicad_pcb (KiCad board)
At the start: 4 copper layers, 257 x 109 mm, 157 parts, among them J1 SFP+, J10 Barrel_Jack, J109 Conn_01x10, J11 Conn_02x06_Odd_Even, J2 SFP+, J209 Conn_01x10, J3 SFP+, J309 Conn_01x10, J4 SFP+, J409 Conn_01x10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

Commit message: Release 2.0-12
Connections:
- net CLK0/CSI0_MCLK renamed CLK0/CSI0_MCLK
- net CLK1/CSI1_MCLK renamed CLK1/CSI1_MCLK
- net SD_CMD/SPI1_DIN renamed SD_CMD/SPI1_DIN
- net SD_DAT0/SPI1_DOUT renamed SD_DAT0/SPI1_DOUT
- net SD_DAT3/SPI1_CS renamed SD_DAT3/SPI1_CS
- net SD_SCLK/SPI1_SCLK renamed SD_SCLK/SPI1_SCLK
- C101 pad 1: +3V3 -> +3.3V
- C102 pad 1: +3V3 -> +3.3V
- C201 pad 1: +3V3 -> +3.3V
- C202 pad 1: +3V3 -> +3.3V
- C301 pad 1: +3V3 -> +3.3V
- C302 pad 1: +3V3 -> +3.3V
- C401 pad 1: +3V3 -> +3.3V
- C402 pad 1: +3V3 -> +3.3V
- C501 pad 1: +3V3 -> +3.3V
- C502 pad 1: +3V3 -> +3.3V
- C601 pad 1: +3V3 -> +3.3V
- C602 pad 1: +3V3 -> +3.3V
- J7 pad 5: +3V3 -> +3.3V
- J7 pad 6: +3V3 -> +3.3V
- J7 pad 9: (no net) -> unconnected-(J7-Pad9)
- L101 pad 1: +3V3 -> +3.3V
- L102 pad 1: +3V3 -> +3.3V
- L201 pad 1: +3V3 -> +3.3V
- L202 pad 1: +3V3 -> +3.3V
- L301 pad 1: +3V3 -> +3.3V
- L302 pad 1: +3V3 -> +3.3V
- L401 pad 1: +3V3 -> +3.3V
- L402 pad 1: +3V3 -> +3.3V
- L501 pad 1: +3V3 -> +3.3V
- L502 pad 1: +3V3 -> +3.3V
- L601 pad 1: +3V3 -> +3.3V
- L602 pad 1: +3V3 -> +3.3V
- P3 pad 10: (no net) -> CSI0_D0-
- P3 pad 60: (no net) -> unconnected-(P3-Pad60)
- P3 pad 8: (no net) -> CSI0_D0+
- P4 pad 1: +3V3 -> +3.3V
- P4 pad 17: +3V3 -> +3.3V
- P5 pad 1: +3V3 -> +3.3V
- P5 pad 17: +3V3 -> +3.3V
- P6 pad 10: (no net) -> unconnected-(P6-Pad10)
- P6 pad 14: (no net) -> unconnected-(P6-Pad14)
- P6 pad 16: (no net) -> unconnected-(P6-Pad16)
- P6 pad 2: (no net) -> unconnected-(P6-Pad2)
- P6 pad 20: (no net) -> unconnected-(P6-Pad20)
- P6 pad 21: (no net) -> unconnected-(P6-Pad21)
- P6 pad 22: (no net) -> unconnected-(P6-Pad22)
- P6 pad 23: (no net) -> unconnected-(P6-Pad23)
- P6 pad 26: (no net) -> unconnected-(P6-Pad26)
- P6 pad 27: (no net) -> unconnected-(P6-Pad27)
- P6 pad 28: (no net) -> unconnected-(P6-Pad28)
- P6 pad 29: (no net) -> unconnected-(P6-Pad29)
- P6 pad 33: (no net) -> unconnected-(P6-Pad33)
- P6 pad 35: (no net) -> unconnected-(P6-Pad35)
- P6 pad 39: (no net) -> unconnected-(P6-Pad39)
- P6 pad 4: (no net) -> unconnected-(P6-Pad4)
- P6 pad 41: (no net) -> unconnected-(P6-Pad41)
- P6 pad 42: (no net) -> unconnected-(P6-Pad42)
- P6 pad 44: (no net) -> unconnected-(P6-Pad44)
- P6 pad 45: (no net) -> unconnected-(P6-Pad45)
- P6 pad 47: (no net) -> unconnected-(P6-Pad47)
- P6 pad 48: (no net) -> unconnected-(P6-Pad48)
- P6 pad 50: (no net) -> unconnected-(P6-Pad50)
- P6 pad 54: (no net) -> unconnected-(P6-Pad54)
- P6 pad 56: (no net) -> unconnected-(P6-Pad56)
- P6 pad 60: (no net) -> unconnected-(P6-Pad60)
- P6 pad 8: (no net) -> unconnected-(P6-Pad8)
- R101 pad 1: +3V3 -> +3.3V
- R102 pad 1: +3V3 -> +3.3V
- R103 pad 1: +3V3 -> +3.3V
- R104 pad 1: +3V3 -> +3.3V
- R105 pad 1: +3V3 -> +3.3V
- R201 pad 1: +3V3 -> +3.3V
- R202 pad 1: +3V3 -> +3.3V
- R203 pad 1: +3V3 -> +3.3V
- R204 pad 1: +3V3 -> +3.3V
- R205 pad 1: +3V3 -> +3.3V
- R301 pad 1: +3V3 -> +3.3V
- R302 pad 1: +3V3 -> +3.3V
- R303 pad 1: +3V3 -> +3.3V
- R304 pad 1: +3V3 -> +3.3V
- R305 pad 1: +3V3 -> +3.3V
- R401 pad 1: +3V3 -> +3.3V
- R402 pad 1: +3V3 -> +3.3V
- R403 pad 1: +3V3 -> +3.3V
- R404 pad 1: +3V3 -> +3.3V
- R405 pad 1: +3V3 -> +3.3V
- R5 pad 1: +3V3 -> +3.3V
- R501 pad 1: +3V3 -> +3.3V
- R502 pad 1: +3V3 -> +3.3V
- R503 pad 1: +3V3 -> +3.3V
- R504 pad 1: +3V3 -> +3.3V
- R505 pad 1: +3V3 -> +3.3V
- R6 pad 1: +3V3 -> +3.3V
- R601 pad 1: +3V3 -> +3.3V
- R602 pad 1: +3V3 -> +3.3V
- R603 pad 1: +3V3 -> +3.3V
- R604 pad 1: +3V3 -> +3.3V
- R605 pad 1: +3V3 -> +3.3V
- R7 pad 1: +3V3 -> +3.3V
- U1 pad A1: (no net) -> unconnected-(U1-PadA1)
- U1 pad A4: (no net) -> unconnected-(U1-PadA4)
- U1 pad A5: (no net) -> unconnected-(U1-PadA5)
- U1 pad B2: (no net) -> unconnected-(U1-PadB2)
- U1 pad B5: (no net) -> unconnected-(U1-PadB5)
- U1 pad C1: +3V3 -> +3.3V
- U1 pad C2: (no net) -> unconnected-(U1-PadC2)
- U1 pad D1: +3V3 -> +3.3V
- U1 pad D2: +3V3 -> +3.3V
- U1 pad E1: +3V3 -> +3.3V
- U1 pad E2: +3V3 -> +3.3V
Routing:
- net +3.3V: track 0.00 -> 359.0 mm, vias 0 -> 57
- net +3V3: track 359.0 -> 0.00 mm, vias 57 -> 0
- added copper zone on F.Cu, net +3.3V
- added copper zone on In2.Cu, net +3.3V
- removed copper zone on F.Cu, net +3V3
- removed copper zone on In2.Cu, net +3V3
Other:
- net class Default removed
- net class Power removed
- net class Thin removed
- board text added: "12"
- board text removed: "11"

Commit message: Release 2.0-13
Parts:
- R1, R2: footprint Capacitor_SMD:C_0402_1005Metric -> Resistor_SMD:R_0402_1005Metric
Connections:
- C9 pad 1: +3V3 -> +3.3V
- REF** pad 1: CHASSIS -> (no net) (x2)
Other:
- board text added: "13"
- board text removed: "12"

Commit message: Release 2.1
Parts:
- added R10: 7K15, Resistor_SMD:R_0402_1005Metric, F.Cu at (82.6, 71.5)
- added R9: 10K, Resistor_SMD:R_0402_1005Metric, F.Cu at (81.4, 71.5)
Connections:
- J9 pad 1: GND -> /ENABLE_RPI_5V
Routing:
- net /ENABLE_RPI_5V: track 0.00 -> 6.87 mm
- net GND: track 1529.8 -> 1535.8 mm, vias 163 -> 162
- net +3V3: track 0.00 -> 0.79 mm, vias 0 -> 1
Other:
- board text added: "spark ver. 2.1"
- board text removed: "13"
- board text removed: ":"
- board text removed: "P/N"
- board text removed: "REV"
- board text removed: "SPARK-V2"
Changed lines of the file:
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@@
   (paper "A4")
   (title_block
-    (title "Spark v.2, (96Boards extension connector 6x SFP+)")
-    (rev "13")
+    (title "Spark ver. 2.1, (96Boards extension connector 6x SFP+)")
     (company "Lightside Instruments AS")
   )
@@
   (net 234 "unconnected-(P6-Pad4)")
   (net 235 "unconnected-(P6-Pad2)")
+  (net 236 "/ENABLE_RPI_5V")
+  (net 237 "+3V3")
   (footprint "spark:molex-sfp-plus-747540-101" (layer "F.Cu")
     (at 157 109 90)
@@
     (fp_line (start 5 10.75) (end -3 10.75) (layer "F.SilkS") (width 0.15))
     (pad "1" smd rect locked (at -1.65 0) (size 0.89 2.1) (layers "F.Cu" "F.Paste" "F.Mask")
-      (net 2 "GND") (pinfunction "Pin_1") (pintype "passive"))
+      (net 236 "/ENABLE_RPI_5V") (pinfunction "Pin_1") (pintype "passive"))
     (pad "2" smd rect locked (at 3.65 0) (size 0.89 2.1) (layers "F.Cu" "F.Paste" "F.Mask")
       (net 10 "SYS_DCIN") (pinfunction "Pin_2") (pintype "passive"))
@@
     )
   )
+  (footprint "Resistor_SMD:R_0402_1005Metric" (layer "F.Cu")
+    (at 81.4 71.5 -90)
+    (descr "Resistor SMD 0402 (1005 Metric), square (rectangular) end terminal, IPC_7351 nominal, (Body size source: IPC-SM-782 page 72, https://www.pcb-3d.com/wordpress/wp-content/uploads/ipc-sm-782a_amendment_1_and_2.pdf), generated with kicad-footprint-generator")
+    (tags "resistor")
+    (property "Sheetfile" "spark.kicad_sch")
+    (property "Sheetname" "")
+    (attr smd)
+    (fp_text reference "R9" (at -2.5 -1.2 90) (layer "F.SilkS")
+      (effects (font (size 1 1) (thickness 0.15)))
+    )
+    (fp_text value "10K" (at 0 1.17 90) (layer "F.Fab")
+      (effects (font (size 1 1) (thickness 0.15)))
+    )
+    (fp_text user "${REFERENCE}" (at 0 0 90) (layer "F.Fab")
+      (effects (font (size 0.26 0.26) (thickness 0.04)))
+    )
+    (fp_line (start -0.153641 0.38) (end 0.153641 0.38) (layer "F.SilkS") (width 0.12))
+    (fp_line (start -0.153641 -0.38) (end 0.153641 -0.38) (layer "F.SilkS") (width 0.12))
+    (fp_line (start 0.93 0.47) (end -0.93 0.47) (layer "F.CrtYd") (width 0.05))
+    (fp_line (start -0.93 0.47) (end -0.93 -0.47) (layer "F.CrtYd") (width 0.05))
+    (fp_line (start -0.93 -0.47) (end 0.93 -0.47) (layer "F.CrtYd") (width 0.05))
+    (fp_line (start 0.93 -0.47) (end 0.93 0.47) (layer "F.CrtYd") (width 0.05))
+    (fp_line (start 0.525 -0.27) (end 0.525 0.27) (layer "F.Fab") (width 0.1))
+    (fp_line (start -0.525 -0.27) (end 0.525 -0.27) (layer "F.Fab") (width 0.1))
+    (fp_line (start -0.525 0.27) (end -0.525 -0.27) (layer "F.Fab") (width 0.1))
+    (fp_line (start 0.525 0.27) (end -0.525 0.27) (layer "F.Fab") (width 0.1))
+    (pad "1" smd roundrect (at -0.51 0 270) (size 0.54 0.64) (layers "F.Cu" "F.Paste" "F.Mask") (roundrect_rratio 0.25)
+      (net 237 "+3V3") (pintype "passive"))
+    (pad "2" smd roundrect (at 0.51 0 270) (size 0.54 0.64) (layers "F.Cu" "F.Paste" "F.Mask") (roundrect_rratio 0.25)
+      (net 236 "/ENABLE_RPI_5V") (pintype "passive"))
+    (model "${KICAD6_3DMODEL_DIR}/Resistor_SMD.3dshapes/R_0402_1005Metric.wrl"
+      (offset (xyz 0 0 0))
+      (scale (xyz 1 1 1))
+      (rotate (xyz 0 0 0))
+    )
+  )
   (footprint "spark:mount_hole" locked (layer "F.Cu")
     (at 250 45)
@@
     )
   )
+  (footprint "Resistor_SMD:R_0402_1005Metric" (layer "F.Cu")
+    (at 82.6 71.5 90)
+    (descr "Resistor SMD 0402 (1005 Metric), square (rectangular) end terminal, IPC_7351 nominal, (Body size source: IPC-SM-782 page 72, https://www.pcb-3d.com/wordpress/wp-content/uploads/ipc-sm-782a_amendment_1_and_2.pdf), generated with kicad-footprint-generator")
+    (tags "resistor")
+    (property "Sheetfile" "spark.kicad_sch")
+    (property "Sheetname" "")
+    (attr smd)
+    (fp_text reference "R10" (at 3 -1.4 90) (layer "F.SilkS")
+      (effects (font (size 1 1) (thickness 0.15)))
+    )
+    (fp_text value "7K15" (at 0 1.17 90) (layer "F.Fab")
+      (effects (font (size 1 1) (thickness 0.15)))
+    )
+    (fp_text user "${REFERENCE}" (at 0 0 90) (layer "F.Fab")
+      (effects (font (size 0.26 0.26) (thickness 0.04)))
+    )
+    (fp_line (start -0.153641 -0.38) (end 0.153641 -0.38) (layer "F.SilkS") (width 0.12))
+    (fp_line (start -0.153641 0.38) (end 0.153641 0.38) (layer "F.SilkS") (width 0.12))
+    (fp_line (start 0.93 0.47) (end -0.93 0.47) (layer "F.CrtYd") (width 0.05))
+    (fp_line (start 0.93 -0.47) (end 0.93 0.47) (layer "F.CrtYd") (width 0.05))
+    (fp_line (start -0.93 -0.47) (end 0.93 -0.47) (layer "F.CrtYd") (width 0.05))
+    (fp_line (start -0.93 0.47) (end -0.93 -0.47) (layer "F.CrtYd") (width 0.05))
+    (fp_line (start -0.525 0.27) (end -0.525 -0.27) (layer "F.Fab") (width 0.1))
+    (fp_line (start 0.525 -0.27) (end 0.525 0.27) (layer "F.Fab") (width 0.1))
+    (fp_line (start 0.525 0.27) (end -0.525 0.27) (layer "F.Fab") (width 0.1))
+    (fp_line (start -0.525 -0.27) (end 0.525 -0.27) (layer "F.Fab") (width 0.1))
+    (pad "1" smd roundrect (at -0.51 0 90) (size 0.54 0.64) (layers "F.Cu" "F.Paste" "F.Mask") (roundrect_rratio 0.25)
+      (net 236 "/ENABLE_RPI_5V") (pintype "passive"))
+    (pad "2" smd roundrect (at 0.51 0 90) (size 0.54 0.64) (layers "F.Cu" "F.Paste" "F.Mask") (roundrect_rratio 0.25)
+      (net 2 "GND") (pintype "passive"))
+    (model "${KICAD6_3DMODEL_DIR}/Resistor_SMD.3dshapes/R_0402_1005Metric.wrl"
+      (offset (xyz 0 0 0))
+      (scale (xyz 1 1 1))
+      (rotate (xyz 0 0 0))
+    )
+  )
   (footprint "LED_SMD:LED_0402_1005Metric" (layer "F.Cu")
     (at 80.2 104.2 -90)
@@
   (gr_line (start 16 150) (end 273 150) (layer "Edge.Cuts") (width 0.1))
   (gr_line (start 16 41) (end 16 150) (layer "Edge.Cuts") (width 0.1))
-  (gr_text "P/N" (at 70.4 62.3) (layer "F.SilkS")
-    (effects (font (size 1.5 1.5) (thickness 0.3)) (justify right))
-  )
-  (gr_text "REV" (at 69.9 65) (layer "F.SilkS")
+  (gr_text "spark ver. 2.1" (at 38.8 81.2) (layer "F.SilkS")
     (effects (font (size 1.5 1.5) (thickness 0.3)) (justify right))
   )
-  (gr_text "SPARK-V2" (at 79.5 62.3) (layer "F.SilkS")
-    (effects (font (size 1.5 1.5) (thickness 0.3)))
-  )
   (gr_text "RPI_5V" (at 92.5 57.5) (layer "F.SilkS")
     (effects (font (size 0.5 0.5) (thickness 0.1)))
   )
-  (gr_text ":" (at 71.5 64.7) (layer "F.SilkS")
-    (effects (font (size 1.5 1.5) (thickness 0.3)))
-  )
-  (gr_text "13" (at 74.5 64.9) (layer "F.SilkS")
-    (effects (font (size 1.5 1.5) (thickness 0.3)))
-  )
-  (gr_text ":" (at 71.5 62.1) (layer "F.SilkS")
-    (effects (font (size 1.5 1.5) (thickness 0.3)))
-  )
   (dimension (type aligned) (layer "B.Fab")
     (pts (xy 273 137.75) (xy 251.85 137.75))
@@
   (segment (start 241.298641 134.799999) (end 240.949999 134.799999) (width 0.254) (layer "F.Cu") (net 2))
   (segment (start 70.2 51.315) (end 69.534801 50.649801) (width 0.254) (layer "F.Cu") (net 2))
-  (segment (start 90 72.65) (end 90 71) (width 0.635) (layer "F.Cu") (net 2))
   (segment (start 231.85 133.6) (end 232.75 134.5) (width 0.381) (layer "F.Cu") (net 2))
   (segment (start 83.6 109.85) (end 83.5 109.75) (width 0.254) (layer "F.Cu") (net 2))
@@
   (segment (start 263.5 89.9) (end 263.5 88.85) (width 0.4) (layer "F.Cu") (net 2))
   (segment (start 92 49.35) (end 92 51) (width 0.635) (layer "F.Cu") (net 2))
-  (segment (start 88 72.65) (end 88 71) (width 0.635) (layer "F.Cu") (net 2))
   (segment (start 219.73 44.365) (end 220.365 45) (width 0.381) (layer "F.Cu") (net 2))
   (segment (start 224.5 92) (end 224.5 93.15) (width 0.4) (layer "F.Cu") (net 2))
@@
   (segment (start 114.68 42) (end 117.22 42) (width 0.635) (layer "F.Cu") (net 2))
   (segment (start 242.25 54.25) (end 242.25 55.504) (width 0.254) (layer "F.Cu") (net 2))
+  (segment (start 82.6 70.99) (end 89.59 70.99) (width 0.254) (layer "F.Cu") (net 2))
   (segment (start 158 111.1) (end 158 109.75) (width 0.381) (layer "F.Cu") (net 2))
   (segment (start 81.6 119.3) (end 81.2 119.3) (width 0.381) (layer "F.Cu") (net 2))
@@
   (segment (start 65.431 119.3) (end 65.5 119.369) (width 0.381) (layer "F.Cu") (net 2))
   (segment (start 232.65 56.4) (end 232.65 54.25) (width 0.254) (layer "F.Cu") (net 2))
+  (segment (start 90 71.4) (end 90 71) (width 0.635) (layer "F.Cu") (net 2))
   (segment (start 201.95 44.365) (end 202.585 45) (width 0.381) (layer "F.Cu") (net 2))
   (segment (start 70.2 47.4) (end 70.2 48) (width 0.254) (layer "F.Cu") (net 2))
@@
   (segment (start 242.25 55.504) (end 242.25 56.5) (width 0.254) (layer "F.Cu") (net 2))
   (segment (start 245.13 47.525) (end 244.125 47.525) (width 0.635) (layer "F.Cu") (net 2))
+  (segment (start 90 72.65) (end 90 71.4) (width 0.635) (layer "F.Cu") (net 2))
+  (segment (start 89.59 70.99) (end 90 71.4) (width 0.254) (layer "F.Cu") (net 2))
   (segment (start 224.05 97.75) (end 224 97.8) (width 0.635) (layer "F.Cu") (net 2))
   (segment (start 242.25 136.75) (end 242.25 135.751358) (width 0.254) (layer "F.Cu") (net 2))
@@
   (via (at 86 109.75) (size 0.6) (drill 0.4) (layers "F.Cu" "B.Cu") (net 2))
   (via (at 98 71) (size 0.6) (drill 0.4) (layers "F.Cu" "B.Cu") (net 2))
-  (via (at 88 71) (size 0.6) (drill 0.4) (layers "F.Cu" "B.Cu") (net 2))
   (via (at 89.3 111.1) (size 0.6) (drill 0.4) (layers "F.Cu" "B.Cu") (net 2))
   (via (at 46.7 113.9) (size 0.6) (drill 0.4) (layers "F.Cu" "B.Cu") (net 2))
@@
   (via (at 251.85 52) (size 0.6) (drill 0.4) (layers "F.Cu" "B.Cu") (net 208))
   (segment (start 251.85 52) (end 251.85 138.99) (width 0.254) (layer "B.Cu") (net 208))
+  (segment (start 83.24 72.65) (end 82.6 72.01) (width 0.254) (layer "F.Cu") (net 236))
+  (segment (start 81.4 72.01) (end 82.6 72.01) (width 0.254) (layer "F.Cu") (net 236))
+  (segment (start 88 72.65) (end 83.24 72.65) (width 0.254) (layer "F.Cu") (net 236))
+  (segment (start 81.4 70.99) (end 81.4 70.2) (width 0.254) (layer "F.Cu") (net 237))
+  (via (at 81.4 70.2) (size 0.6) (drill 0.4) (layers "F.Cu" "B.Cu") (net 237))
   (zone (net 47) (net_name "+3.3V") (layer "F.Cu") (hatch edge 0.508)
     (priority 2)

Commit message: Release 2.2
Parts:
- removed J7: PTH08T221W, spark:R-PDSS-B11
- removed R8: 1K21, Resistor_SMD:R_0402_1005Metric
- removed SW3: SW_DIP_x01, Connector_PinHeader_2.54mm:PinHeader_1x02_P2.54mm_Vertical
- added J14: Conn_02x07_Odd_Even, Connector_PinSocket_2.00mm:PinSocket_2x07_P2.00mm_Vertical_SMD, F.Cu at (40.0, 70.0)
- added J15: Conn_02x07_Odd_Even, Connector_PinSocket_2.00mm:PinSocket_2x07_P2.00mm_Vertical_SMD, F.Cu at (40.0, 52.0)
- J11, J9: value Conn_02x06_Odd_Even -> Conn_02x07_Odd_Even; footprint spark:Socket_Strip_SMD_2x6_Pitch2mm -> Connector_PinSocket_2.00mm:PinSocket_2x07_P2.00mm_Vertical_SMD
- REF**: footprint spark:96Boards_CE_outline_std_brick_top -> spark:96Boards_CE_outline_std_brick_corner
- moved ? 5.10 mm to (50.0, 79.0)
- moved J11 4.12 mm to (92.0, 52.0)
- moved J9 4.12 mm to (92.0, 70.0)
- moved R10 2.00 mm to (80.6, 71.5)
- moved R9 2.00 mm to (79.4, 71.5)
Connections:
- net Net-(P4-Pad11) renamed ENABLE_3.3V
- J11 pad 1: RPI_5V -> RPI_I2C_SCL
- J11 pad 10: GND -> RPI_5V
- J11 pad 11: RPI_5V -> GND
- J11 pad 12: GND -> RPI_5V
- J11 pad 2: GND -> RPI_I2C_SDA
- J11 pad 3: RPI_5V -> GND
- J11 pad 4: GND -> RPI_5V
- J11 pad 5: RPI_5V -> GND
- J11 pad 6: GND -> RPI_5V
- J11 pad 7: RPI_5V -> GND
- J11 pad 8: GND -> RPI_5V
- J11 pad 9: RPI_5V -> GND
- J9 pad 1: /ENABLE_RPI_5V -> unconnected-(J9-Pad1)
- J9 pad 10: SYS_DCIN -> GND
- J9 pad 11: GND -> SYS_DCIN
- J9 pad 12: SYS_DCIN -> GND
- J9 pad 2: SYS_DCIN -> /ENABLE_RPI_5V
- J9 pad 3: GND -> SYS_DCIN
- J9 pad 4: SYS_DCIN -> GND
- J9 pad 5: GND -> SYS_DCIN
- J9 pad 6: SYS_DCIN -> GND
- J9 pad 7: GND -> SYS_DCIN
- J9 pad 8: SYS_DCIN -> GND
- J9 pad 9: GND -> SYS_DCIN
- P4 pad 3: RPI_I2C_SDA -> RPI_I2C_SCL
- P4 pad 5: RPI_I2C_SCL -> RPI_I2C_SDA
- P5 pad 3: RPI_I2C_SDA -> RPI_I2C_SCL
- P5 pad 5: RPI_I2C_SCL -> RPI_I2C_SDA
Routing:
- net RPI_I2C_SDA: track 144.6 -> 248.5 mm, vias 4 -> 8
- net ENABLE_3.3V: track 105.7 -> 205.6 mm
- net RPI_I2C_SCL: track 151.2 -> 250.6 mm, vias 4 -> 8
- net RPI_5V: track 216.7 -> 226.6 mm
- net +3.3V: track 359.0 -> 368.9 mm, vias 57 -> 63
- net GND: track 1535.8 -> 1526.6 mm, vias 162 -> 174
- net Net-(J7-Pad11): track 7.61 -> 0.00 mm
- net Net-(J7-Pad8): track 5.30 -> 0.00 mm
- net SYS_DCIN: vias 14 -> 20
Other:
- board text added: ".2"
- board text added: "3.3V"
- board text added: "spark-2"
- board text removed: "spark ver. 2.1"

Commit message: Release 2.2-1
Connections:
- R9 pad 1: +3V3 -> +3.3V
Routing:
- net +3.3V: track 368.9 -> 369.7 mm, vias 63 -> 64
- net +3V3: track 0.79 -> 0.00 mm, vias 1 -> 0
Other:
- board text added: "-1"
Changed lines of the file:
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@@
   (paper "A4")
   (title_block
-    (title "Spark ver. 2.2, (96Boards extension connector 6x SFP+)")
+    (title "Spark ver. 2.2-1, (96Boards extension connector 6x SFP+)")
     (company "Lightside Instruments AS")
   )
@@
   (net 231 "unconnected-(P6-Pad2)")
   (net 232 "/ENABLE_RPI_5V")
-  (net 233 "+3V3")
+  (net 233 "+3.3V")
   (net 234 "unconnected-(J9-Pad1)")
   (net 235 "unconnected-(J14-Pad1)")
@@
     (fp_line (start 0.525 0.27) (end -0.525 0.27) (layer "F.Fab") (width 0.1))
     (pad "1" smd roundrect (at -0.51 0 270) (size 0.54 0.64) (layers "F.Cu" "F.Paste" "F.Mask") (roundrect_rratio 0.25)
-      (net 233 "+3V3") (pintype "passive"))
+      (net 233 "+3.3V") (pintype "passive"))
     (pad "2" smd roundrect (at 0.51 0 270) (size 0.54 0.64) (layers "F.Cu" "F.Paste" "F.Mask") (roundrect_rratio 0.25)
       (net 232 "/ENABLE_RPI_5V") (pintype "passive"))
@@
     (effects (font (size 3 3) (thickness 0.75)) (justify right))
   )
+  (gr_text "-1" (at 41.2 84.9) (layer "F.SilkS")
+    (effects (font (size 3 3) (thickness 0.75)) (justify left))
+  )
   (gr_text "3.3V" (at 40 60) (layer "F.SilkS")

Commit message: Release 2.2-2
Other:
- board text added: "-2"
- board text removed: "-1"
Changed lines of the file:
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@@
   (paper "A4")
   (title_block
-    (title "Spark ver. 2.2-1, (96Boards extension connector 6x SFP+)")
+    (title "Spark ver. 2.2-2, (96Boards extension connector 6x SFP+)")
     (company "Lightside Instruments AS")
   )
@@
     (property "Sheetname" "")
     (attr smd)
-    (fp_text reference "D101" (at 0 -1.17 -90) (layer "F.SilkS")
+    (fp_text reference "D101" (at 0 1.1 -90) (layer "F.SilkS")
       (effects (font (size 1 1) (thickness 0.15)))
     )
@@
     (effects (font (size 3 3) (thickness 0.75)) (justify right))
   )
-  (gr_text "-1" (at 41.2 84.9) (layer "F.SilkS")
+  (gr_text "-2" (at 41.2 84.9) (layer "F.SilkS")
     (effects (font (size 3 3) (thickness 0.75)) (justify left))
   )
