File: board/spark.kicad_pcb (KiCad board)
At the start: 4 copper layers, 257 x 109 mm, 158 parts, among them J1 SFP+, J10 Barrel_Jack, J109 Conn_01x10, J11 Conn_02x07_Odd_Even, J14 Conn_02x07_Odd_Even, J15 Conn_02x07_Odd_Even, J2 SFP+, J209 Conn_01x10, J3 SFP+, J309 Conn_01x10, J4 SFP+, J409 Conn_01x10, J5 SFP+, J509 Conn_01x10, J6 SFP+, J609 Conn_01x10, J8 Conn_02x30_Odd_Even, J9 Conn_02x07_Odd_Even, P1 CONN_02X20, P2 Conn_02x20_Odd_Even, P3 CONN_02X30, P4 Conn_02x20_Odd_Even, P5 Conn_02x20_Odd_Even, P6 CONN_02X30, SW1 SW_Push, SW2 SW_DIP_x06, SW4 SW_DIP_x01, U1 LTM4624IYPBF, U2 PCA9306

Commit message: Release 2.2-6
Other:
- board text added: "-6"
- board text removed: "-2"
Changed lines of the file:
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@@
 	(paper "A4")
 	(title_block
-		(title "Spark ver. 2.2-2, (96Boards extension connector 6x SFP+)")
+		(title "Spark ver. 2.2-6, (96Boards extension connector 6x SFP+)")
 		(company "Lightside Instruments AS")
 	)
@@
 		)
 	)
-	(gr_text "-2"
+	(gr_text "-6"
 		(at 41.2 84.9 0)
 		(layer "F.SilkS")
