File: board/spark.kicad_sch (KiCad schematic)
At the start: 143 parts, among them J1 SFP+, J10 Barrel_Jack, J109 Conn_01x10, J11 Conn_02x06_Odd_Even, J2 SFP+, J209 Conn_01x10, J3 SFP+, J309 Conn_01x10, J4 SFP+, J409 Conn_01x10, J5 SFP+, J509 Conn_01x10, J6 SFP+, J609 Conn_01x10, J7 PTH08T221W, J8 Conn_02x30_Odd_Even, J9 Conn_02x06_Odd_Even, P1 CONN_02X20, P2 Conn_02x20_Odd_Even, P3 CONN_02X30, P4 Conn_02x20_Odd_Even, P5 Conn_02x20_Odd_Even, P6 CONN_02X30, SW1 SW_Push, SW2 SW_DIP_x06, SW3 SW_DIP_x01, SW4 SW_DIP_x01, U1 LTM4624IYPBF, U2 PCA9306

Commit message: Release 2.0-13
Parts:
- C7, C9: symbol Device:CP -> Device:C_Polarized
- D102, D202, D302, D402, D502, D602: symbol Device:LED -> Device:LED_Filled
- R1, R2: footprint Capacitor_SMD:C_0402_1005Metric -> Resistor_SMD:R_0402_1005Metric
Connections:
- net +3.3V: now also C9.1
- net GND: now also C7.2, C9.2
- net SYS_DCIN: now also C7.1
Changed lines of the file:
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@@
   (title_block
     (title "Spark v.2 - 96Boards extension connector 6x SFP+")
-    (rev "12")
+    (rev "13")
     (company "Lightside Instruments AS")
   )
@@
     (pin "2")
   )
-  (symbol (lib_id "Device:CP") (at 151.13 273.05 0) (unit 1)
+  (symbol (lib_id "Device:C_Polarized") (at 151.13 273.05 0) (unit 1)
     (in_bom yes) (on_board yes)
     (property "Reference" "C7" (id 0) (at 154.1272 271.8816 0)
@@
       (effects (font (size 1.27 1.27)) hide)
     )
-    (property "Datasheet" "" (id 3) (at 151.13 273.05 0)
+    (property "Datasheet" "~" (id 3) (at 151.13 273.05 0)
       (effects (font (size 1.27 1.27)) hide)
     )
+    (pin "1")
+    (pin "2")
   )
   (symbol (lib_id "power:GND") (at 151.13 276.86 0) (unit 1)
@@
     (pin "1")
   )
-  (symbol (lib_id "Device:CP") (at 212.09 280.67 0) (unit 1)
+  (symbol (lib_id "Device:C_Polarized") (at 212.09 280.67 0) (unit 1)
     (in_bom yes) (on_board yes)
     (property "Reference" "C9" (id 0) (at 215.0872 279.5016 0)
@@
       (effects (font (size 1.27 1.27)) hide)
     )
+    (pin "1")
+    (pin "2")
   )
   (symbol (lib_id "power:GND") (at 212.09 284.48 0) (unit 1)
@@
     (pin "2")
   )
-  (symbol (lib_id "Device:LED") (at 49.53 185.42 90) (unit 1)
+  (symbol (lib_id "Device:LED_Filled") (at 49.53 185.42 90) (unit 1)
     (in_bom yes) (on_board yes)
     (property "Reference" "D102" (id 0) (at 52.5272 184.4548 90)
@@
     (pin "2")
   )
-  (symbol (lib_id "Device:LED") (at 171.45 186.69 90) (unit 1)
+  (symbol (lib_id "Device:LED_Filled") (at 171.45 186.69 90) (unit 1)
     (in_bom yes) (on_board yes)
     (property "Reference" "D202" (id 0) (at 174.4472 185.7248 90)
@@
     (pin "2")
   )
-  (symbol (lib_id "Device:LED") (at 293.37 186.69 90) (unit 1)
+  (symbol (lib_id "Device:LED_Filled") (at 293.37 186.69 90) (unit 1)
     (in_bom yes) (on_board yes)
     (property "Reference" "D302" (id 0) (at 296.3672 185.7248 90)
@@
     (pin "2")
   )
-  (symbol (lib_id "Device:LED") (at 415.29 186.69 90) (unit 1)
+  (symbol (lib_id "Device:LED_Filled") (at 415.29 186.69 90) (unit 1)
     (in_bom yes) (on_board yes)
     (property "Reference" "D402" (id 0) (at 418.2872 185.7248 90)
@@
     (pin "2")
   )
-  (symbol (lib_id "Device:LED") (at 537.21 186.69 90) (unit 1)
+  (symbol (lib_id "Device:LED_Filled") (at 537.21 186.69 90) (unit 1)
     (in_bom yes) (on_board yes)
     (property "Reference" "D502" (id 0) (at 540.2072 185.7248 90)
@@
     (pin "2")
   )
-  (symbol (lib_id "Device:LED") (at 659.13 186.69 90) (unit 1)
+  (symbol (lib_id "Device:LED_Filled") (at 659.13 186.69 90) (unit 1)
     (in_bom yes) (on_board yes)
     (property "Reference" "D602" (id 0) (at 662.1272 185.7248 90)
@@
       (effects (font (size 1.27 1.27)) (justify left))
     )
-    (property "Footprint" "Capacitor_SMD:C_0402_1005Metric" (id 2) (at 155.702 367.03 90)
+    (property "Footprint" "Resistor_SMD:R_0402_1005Metric" (id 2) (at 155.702 367.03 90)
       (effects (font (size 1.27 1.27)) hide)
     )
@@
     (property "Reference" "R1" (id 0) (at 151.13 342.7222 90))
     (property "Value" "13K3" (id 1) (at 151.13 345.0336 90))
-    (property "Footprint" "Capacitor_SMD:C_0402_1005Metric" (id 2) (at 151.13 346.202 90)
+    (property "Footprint" "Resistor_SMD:R_0402_1005Metric" (id 2) (at 151.13 346.202 90)
       (effects (font (size 1.27 1.27)) hide)
     )
@@
     )
     (path "/00000000-0000-0000-0000-00006100cf67"
-      (reference "R1") (unit 1) (value "13K3") (footprint "Capacitor_SMD:C_0402_1005Metric")
+      (reference "R1") (unit 1) (value "13K3") (footprint "Resistor_SMD:R_0402_1005Metric")
     )
     (path "/00000000-0000-0000-0000-0000607cdf30"
-      (reference "R2") (unit 1) (value "10K") (footprint "Capacitor_SMD:C_0402_1005Metric")
+      (reference "R2") (unit 1) (value "10K") (footprint "Resistor_SMD:R_0402_1005Metric")
     )
     (path "/00000000-0000-0000-0000-00006134158a"

Commit message: Release 2.1
Parts:
- added R10: 7K15, Resistor_SMD:R_0402_1005Metric, symbol Device:R
- added R9: 10K, Resistor_SMD:R_0402_1005Metric, symbol Device:R
Connections:
- net GND: now also R10.2; no longer J9.1 (Pin_1)
- new net +3V3: R9.1
- new net ENABLE_RPI_5V: J9.1 (Pin_1), R10.1, R9.2
Other:
- title: Spark v.2 - 96Boards extension connector 6x SFP+ -> spark-2.1 - 96Boards extension connector 6x SFP+
Changed lines of the file:
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@@
   (paper "A0")
   (title_block
-    (title "Spark v.2 - 96Boards extension connector 6x SFP+")
-    (rev "13")
+    (title "spark-2.1 - 96Boards extension connector 6x SFP+")
     (company "Lightside Instruments AS")
   )
@@
   (junction (at 80.01 134.62) (diameter 0) (color 0 0 0 0)
   )
+  (junction (at 267.97 308.61) (diameter 0) (color 0 0 0 0)
+  )
   (junction (at 297.18 67.31) (diameter 0) (color 0 0 0 0)
   )
@@
   (junction (at 196.85 135.89) (diameter 0) (color 0 0 0 0)
   )
-  (junction (at 260.35 332.74) (diameter 0) (color 0 0 0 0)
-  )
   (junction (at 444.5 260.35) (diameter 0) (color 0 0 0 0)
   )
@@
     (stroke (width 0) (type default) (color 0 0 0 0))
   )
-  (wire (pts (xy 260.35 330.2) (xy 260.35 332.74))
-    (stroke (width 0) (type default) (color 0 0 0 0))
-  )
   (wire (pts (xy 212.09 36.83) (xy 214.63 36.83))
     (stroke (width 0) (type default) (color 0 0 0 0))
@@
     (stroke (width 0) (type default) (color 0 0 0 0))
   )
+  (wire (pts (xy 260.35 308.61) (xy 260.35 330.2))
+    (stroke (width 0) (type default) (color 0 0 0 0))
+  )
   (wire (pts (xy 711.2 160.02) (xy 715.01 160.02))
     (stroke (width 0) (type default) (color 0 0 0 0))
@@
     (stroke (width 0) (type default) (color 0 0 0 0))
   )
+  (wire (pts (xy 267.97 308.61) (xy 260.35 308.61))
+    (stroke (width 0) (type default) (color 0 0 0 0))
+  )
   (wire (pts (xy 280.67 337.82) (xy 280.67 340.36))
     (stroke (width 0) (type default) (color 0 0 0 0))
@@
     (effects (font (size 1.524 1.524)) (justify left bottom))
   )
+  (label "ENABLE_RPI_5V" (at 260.35 308.61 180)
+    (effects (font (size 1.524 1.524)) (justify right bottom))
+  )
   (global_label "DSI_CLK-" (shape bidirectional) (at 474.98 167.64 0) (fields_autoplaced)
     (effects (font (size 1.524 1.524)) (justify left))
@@
   (symbol (lib_id "power:+5VP") (at 109.22 246.38 0) (unit 1)
     (in_bom yes) (on_board yes)
-    (property "Reference" "#PWR?" (id 0) (at 109.22 250.19 0)
+    (property "Reference" "#PWR0193" (id 0) (at 109.22 250.19 0)
       (effects (font (size 1.27 1.27)) hide)
     )
@@
     (pin "1")
   )
+  (symbol (lib_id "Device:R") (at 267.97 312.42 0) (unit 1)
+    (in_bom yes) (on_board yes) (fields_autoplaced)
+    (property "Reference" "R10" (id 0) (at 270.51 311.1499 0)
+      (effects (font (size 1.27 1.27)) (justify left))
+    )
+    (property "Value" "7K15" (id 1) (at 270.51 313.6899 0)
+      (effects (font (size 1.27 1.27)) (justify left))
+    )
+    (property "Footprint" "Resistor_SMD:R_0402_1005Metric" (id 2) (at 266.192 312.42 90)
+      (effects (font (size 1.27 1.27)) hide)
+    )
+    (property "Datasheet" "~" (id 3) (at 267.97 312.42 0)
+      (effects (font (size 1.27 1.27)) hide)
+    )
+    (pin "1")
+    (pin "2")
+  )
+  (symbol (lib_name "+3.3V_1") (lib_id "power:+3.3V") (at 267.97 300.99 0) (unit 1)
+    (in_bom yes) (on_board yes) (fields_autoplaced)
+    (property "Reference" "#PWR0192" (id 0) (at 267.97 304.8 0)
+      (effects (font (size 1.27 1.27)) hide)
+    )
+    (property "Value" "+3.3V" (id 1) (at 267.97 295.91 0))
+    (property "Footprint" "" (id 2) (at 267.97 300.99 0)
+      (effects (font (size 1.27 1.27)) hide)
+    )
+    (property "Datasheet" "" (id 3) (at 267.97 300.99 0)
+      (effects (font (size 1.27 1.27)) hide)
+    )
+    (pin "1")
+  )
+  (symbol (lib_name "GND_1") (lib_id "power:GND") (at 267.97 316.23 0) (unit 1)
+    (in_bom yes) (on_board yes) (fields_autoplaced)
+    (property "Reference" "#PWR0191" (id 0) (at 267.97 322.58 0)
+      (effects (font (size 1.27 1.27)) hide)
+    )
+    (property "Value" "GND" (id 1) (at 267.97 321.31 0))
+    (property "Footprint" "" (id 2) (at 267.97 316.23 0)
+      (effects (font (size 1.27 1.27)) hide)
+    )
+    (property "Datasheet" "" (id 3) (at 267.97 316.23 0)
+      (effects (font (size 1.27 1.27)) hide)
+    )
+    (pin "1")
+  )
+  (symbol (lib_id "Device:R") (at 267.97 304.8 0) (unit 1)
+    (in_bom yes) (on_board yes) (fields_autoplaced)
+    (property "Reference" "R9" (id 0) (at 270.51 303.5299 0)
+      (effects (font (size 1.27 1.27)) (justify left))
+    )
+    (property "Value" "10K" (id 1) (at 270.51 306.0699 0)
+      (effects (font (size 1.27 1.27)) (justify left))
+    )
+    (property "Footprint" "Resistor_SMD:R_0402_1005Metric" (id 2) (at 266.192 304.8 90)
+      (effects (font (size 1.27 1.27)) hide)
+    )
+    (property "Datasheet" "~" (id 3) (at 267.97 304.8 0)
+      (effects (font (size 1.27 1.27)) hide)
+    )
+    (pin "1")
+    (pin "2")
+  )
   (sheet_instances
     (path "/" (page "1"))
@@
       (reference "#PWR0190") (unit 1) (value "GND") (footprint "")
     )
+    (path "/c962e5b0-8a5e-44da-a714-7e52b23ec1a5"
+      (reference "#PWR0191") (unit 1) (value "GND") (footprint "")
+    )
+    (path "/bd133d4c-b28b-4b97-983d-e5f23fff1a2f"
+      (reference "#PWR0192") (unit 1) (value "+3.3V") (footprint "")
+    )
     (path "/00000000-0000-0000-0000-0000629128f7"
-      (reference "#PWR?") (unit 1) (value "+5VP") (footprint "")
+      (reference "#PWR0193") (unit 1) (value "+5VP") (footprint "")
     )
     (path "/00000000-0000-0000-0000-0000611ed4f3"
@@
       (reference "R8") (unit 1) (value "1K21") (footprint "Resistor_SMD:R_0402_1005Metric")
     )
+    (path "/d96ecd7a-8974-4818-a0ad-ef5fdf4a961f"
+      (reference "R9") (unit 1) (value "10K") (footprint "Resistor_SMD:R_0402_1005Metric")
+    )
+    (path "/86d3c04c-25af-4555-95bf-649521c0b9be"
+      (reference "R10") (unit 1) (value "7K15") (footprint "Resistor_SMD:R_0402_1005Metric")
+    )
     (path "/00000000-0000-0000-0000-00005d92e865"

Commit message: Release 2.2
Parts:
- removed J7: PTH08T221W, spark:R-PDSS-B11, symbol spark:PTH08T221W
- removed R8: 1K21, Resistor_SMD:R_0402_1005Metric, symbol Device:R
- removed SW3: SW_DIP_x01, Connector_PinHeader_2.54mm:PinHeader_1x02_P2.54mm_Vertical, symbol Switch:SW_DIP_x01
- added J14, J15: Conn_02x07_Odd_Even, Connector_PinSocket_2.00mm:PinSocket_2x07_P2.00mm_Vertical_SMD, symbol Connector_Generic:Conn_02x07_Odd_Even
- J11, J9: value Conn_02x06_Odd_Even -> Conn_02x07_Odd_Even; footprint spark:Socket_Strip_SMD_2x6_Pitch2mm -> Connector_PinSocket_2.00mm:PinSocket_2x07_P2.00mm_Vertical_SMD; symbol Connector_Generic:Conn_02x06_Odd_Even -> Connector_Generic:Conn_02x07_Odd_Even
Connections:
- net +3.3V: now also J15.10 (Pin_10), J15.12 (Pin_12), J15.14 (Pin_14), J15.4 (Pin_4), J15.6 (Pin_6), J15.8 (Pin_8)
- net +5VP: now also J11.10 (Pin_10), J11.12 (Pin_12), J11.14 (Pin_14), J11.4 (Pin_4), J11.6 (Pin_6), J11.8 (Pin_8); no longer J11.1 (Pin_1), J11.11 (Pin_11), J11.3 (Pin_3), J11.5 (Pin_5), J11.7 (Pin_7), J11.9 (Pin_9)
- net ENABLE_RPI_5V: now also J9.2 (Pin_2); no longer J9.1 (Pin_1)
- net GND: now also J11.11 (Pin_11), J11.13 (Pin_13), J11.3 (Pin_3), J11.5 (Pin_5), J11.7 (Pin_7), J11.9 (Pin_9), J9.10 (Pin_10), J9.12 (Pin_12), J9.14 (Pin_14), J9.4 (Pin_4), J9.6 (Pin_6), J9.8 (Pin_8), J14.10 (Pin_10), J14.12 (Pin_12), J14.14 (Pin_14), J14.4 (Pin_4), J14.6 (Pin_6), J14.8 (Pin_8), J15.11 (Pin_11), J15.13 (Pin_13), J15.3 (Pin_3), J15.5 (Pin_5), J15.7 (Pin_7), J15.9 (Pin_9); no longer J11.10 (Pin_10), J11.12 (Pin_12), J11.2 (Pin_2), J11.4 (Pin_4), J11.6 (Pin_6), J11.8 (Pin_8), J9.11 (Pin_11), J9.3 (Pin_3), J9.5 (Pin_5), J9.7 (Pin_7), J9.9 (Pin_9)
- net RPI_I2C_SCL: now also J11.1 (Pin_1), P4.3 (Pin_3), P5.3 (Pin_3), J15.1 (Pin_1); no longer P4.5 (Pin_5), P5.5 (Pin_5)
- net RPI_I2C_SDA: now also J11.2 (Pin_2), P4.5 (Pin_5), P5.5 (Pin_5), J15.2 (Pin_2); no longer P4.3 (Pin_3), P5.3 (Pin_3)
- net SYS_DCIN: now also J9.11 (Pin_11), J9.13 (Pin_13), J9.3 (Pin_3), J9.5 (Pin_5), J9.7 (Pin_7), J9.9 (Pin_9), J14.11 (Pin_11), J14.13 (Pin_13), J14.3 (Pin_3), J14.5 (Pin_5), J14.7 (Pin_7), J14.9 (Pin_9); no longer J9.10 (Pin_10), J9.12 (Pin_12), J9.2 (Pin_2), J9.4 (Pin_4), J9.6 (Pin_6), J9.8 (Pin_8)
- net ENABLE_3.3V: now reaches P4.11 (Pin_11), P5.11 (Pin_11)
- net ENABLE_3.3V: now also J14.2 (Pin_2)
- no-connect marks 2 -> 4
Other:
- note added: "3.3V Alternative External Power supply connector"
- note added: "3.3V power supply option."
- note removed: "3.3V Power supply"
- note removed: "Alternative 3.3V power supply option."
- title: spark-2.1 - 96Boards extension connector 6x SFP+ -> spark-2.2 - 96Boards extension connector 6x SFP+
- moved on the sheet: C7, C8, C9, R10, R9

Commit message: Release 2.2-1
Other:
- title: spark-2.2 - 96Boards extension connector 6x SFP+ -> spark-2.2-1 - 96Boards extension connector 6x SFP+
Changed lines of the file:
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@@
   (paper "A0")
   (title_block
-    (title "spark-2.2 - 96Boards extension connector 6x SFP+")
+    (title "spark-2.2-1 - 96Boards extension connector 6x SFP+")
     (company "Lightside Instruments AS")
   )

Commit message: Release 2.2-2
Other:
- title: spark-2.2-1 - 96Boards extension connector 6x SFP+ -> spark-2.2-2 - 96Boards extension connector 6x SFP+
Changed lines of the file:
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@@
   (paper "A0")
   (title_block
-    (title "spark-2.2-1 - 96Boards extension connector 6x SFP+")
+    (title "spark-2.2-2 - 96Boards extension connector 6x SFP+")
     (company "Lightside Instruments AS")
   )
